File: hog32a.sch (KiCad schematic (older format))
At the start: 43 parts, among them J1 REG:3V3, J10 Conn_01x07, J11 Conn_01x06_Male, J12 dht22, J13 Screw_Terminal_01x02, J14 Conn_01x09_Female, J15 Conn_01x05, J16 LBO, J17 Conn_01x12_Female, J18 Barrel_Jack_Switch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

Commit message: update;
Parts:
- removed J16: LBO, Pin_Headers:Pin_Header_Straight_2x03_Pitch2.54mm, symbol hog32a-rescue:Conn_02x03_Odd_Even
- removed J3: VINS, TerminalBlocks_Phoenix:TerminalBlock_Phoenix_PT-3.5mm_2pol, symbol hog32a-rescue:Conn_01x02
- added J3: Conn_01x06_Female, Connector_PinHeader_2.54mm:PinHeader_1x06_P2.54mm_Vertical, symbol Connector:Conn_01x06_Female
- BT1: footprint dwb:cr1220 -> Battery:BatteryHolder_Keystone_3000_1x12mm
- J18: footprint dwb:barrel_5.5 -> Connector_BarrelJack:BarrelJack_Horizontal
Connections:
- wire segments 96 -> 101
Other:
- moved on the sheet: J18
Changed lines of the file:
@@
 	1    0    0    -1
 $EndComp
-$Comp
-L hog32a-rescue:Conn_01x02 J3
-U 1 1 5B89258D
-P 1500 1050
-F 0 "J3" H 1500 1150 50  0000 C CNN
-F 1 "VINS" H 1500 850 50  0000 C CNN
-F 2 "TerminalBlocks_Phoenix:TerminalBlock_Phoenix_PT-3.5mm_2pol" H 1500 1050 50  0001 C CNN
-F 3 "" H 1500 1050 50  0001 C CNN
-	1    1500 1050
-	1    0    0    -1
-$EndComp
-Text GLabel 1300 1150 0    60   Input ~ 0
+Text GLabel 10450 3450 2    60   Input ~ 0
 VIN
 $Comp
 L hog32a-rescue:GND #PWR024
 U 1 1 5B89266B
-P 1000 1050
-F 0 "#PWR024" H 1000 800 50  0001 C CNN
-F 1 "GND" H 1000 900 50  0000 C CNN
-F 2 "" H 1000 1050 50  0001 C CNN
-F 3 "" H 1000 1050 50  0001 C CNN
-	1    1000 1050
-	1    0    0    -1
-$EndComp
-Text Notes 1100 800  0    60   ~ 0
+P 10550 3800
+F 0 "#PWR024" H 10550 3550 50  0001 C CNN
+F 1 "GND" H 10550 3650 50  0000 C CNN
+F 2 "" H 10550 3800 50  0001 C CNN
+F 3 "" H 10550 3800 50  0001 C CNN
+	1    10550 3800
+	1    0    0    -1
+$EndComp
+Text Notes 10050 3350 0    60   ~ 0
 Power In
 $Comp
@@
 Text GLabel 9500 5500 0    60   Input ~ 0
 DIO3
-$Comp
-L hog32a-rescue:Conn_02x03_Odd_Even J16
-U 1 1 5B91ABB9
-P 10400 5350
-F 0 "J16" H 10450 5550 50  0000 C CNN
-F 1 "LBO" H 10450 5150 50  0000 C CNN
-F 2 "Pin_Headers:Pin_Header_Straight_2x03_Pitch2.54mm" H 10400 5350 50  0001 C CNN
-F 3 "" H 10400 5350 50  0001 C CNN
-	1    10400 5350
-	0    -1   -1   0
-$EndComp
 Text GLabel 10300 5050 1    60   Input ~ 0
 32
+Text GLabel 10500 5050 1    60   Input ~ 0
+25
+Text GLabel 10700 5050 1    60   Input ~ 0
+27
 Text GLabel 10400 5050 1    60   Input ~ 0
-25
-Text GLabel 10500 5050 1    60   Input ~ 0
-27
-Text GLabel 10300 5550 3    60   Input ~ 0
 33
-Text GLabel 10400 5550 3    60   Input ~ 0
+Text GLabel 10600 5050 1    60   Input ~ 0
 26
-Text GLabel 10500 5550 3    60   Input ~ 0
+Text GLabel 10800 5050 1    60   Input ~ 0
 DIO5
 Text GLabel 6200 1800 0    60   Input ~ 0
@@
 Connection ~ 1350 3650
 Wire Wire Line
-	1000 1050 1300 1050
-Wire Wire Line
 	950  7000 950  7200
 Wire Wire Line
@@
 F 0 "BT1" H 2850 3950 50  0000 L CNN
 F 1 "Battery_Cell" H 2650 3850 50  0000 L CNN
-F 2 "dwb:cr1220" V 3150 3960 50  0001 C CNN
+F 2 "Battery:BatteryHolder_Keystone_3000_1x12mm" V 3150 3960 50  0001 C CNN
 F 3 "~" V 3150 3960 50  0001 C CNN
 	1    3150 3900
@@
 L Connector:Barrel_Jack_Switch J18
 U 1 1 5CED6D12
-P -500 1100
-F 0 "J18" H -445 1417 50  0000 C CNN
-F 1 "Barrel_Jack_Switch" H -445 1326 50  0000 C CNN
-F 2 "dwb:barrel_5.5" H -450 1060 50  0001 C CNN
-F 3 "~" H -450 1060 50  0001 C CNN
-	1    -500 1100
-	1    0    0    -1
+P 10000 3800
+F 0 "J18" H 10055 4117 50  0000 C CNN
+F 1 "Barrel_Jack_Switch" H 10055 4026 50  0000 C CNN
+F 2 "Connector_BarrelJack:BarrelJack_Horizontal" H 10050 3760 50  0001 C CNN
+F 3 "~" H 10050 3760 50  0001 C CNN
+	1    10000 3800
+	1    0    0    -1
+$EndComp
+Wire Wire Line
+	10550 3800 10400 3800
+Wire Wire Line
+	10300 3900 10400 3900
+Wire Wire Line
+	10400 3900 10400 3800
+Connection ~ 10400 3800
+Wire Wire Line
+	10400 3800 10300 3800
+Wire Wire Line
+	10450 3700 10450 3450
+Wire Wire Line
+	10450 3700 10300 3700
+$Comp
+L Connector:Conn_01x06_Female J3
+U 1 1 5CE353BC
+P 10600 5250
+F 0 "J3" V 10447 5498 50  0000 L CNN
+F 1 "Conn_01x06_Female" V 10538 5498 50  0000 L CNN
+F 2 "Connector_PinHeader_2.54mm:PinHeader_1x06_P2.54mm_Vertical" H 10600 5250 50  0001 C CNN
+F 3 "~" H 10600 5250 50  0001 C CNN
+	1    10600 5250
+	0    1    1    0
 $EndComp
 $EndSCHEMATC

Commit message: update
Parts:
- added J16: Conn_01x02_Male, Connector_PinHeader_2.54mm:PinHeader_1x02_P2.54mm_Vertical, symbol Connector:Conn_01x02_Male
- added J19: Screw_Terminal_01x04, TerminalBlock_Phoenix:TerminalBlock_Phoenix_PT-1,5-4-3.5-H_1x04_P3.50mm_Horizontal, symbol Connector:Screw_Terminal_01x04
Connections:
- net +3V3: now also J19.4 (Pin_4)
- net 14:SCL: now also J19.2 (Pin_2)
- net 2:SDA: now also J19.1 (Pin_1)
- net GND: now also J19.3 (Pin_3)
- net RESET: now also J16.1 (Pin_1)
- net at R2.2, U3.5 (DRV): now also J16.2 (Pin_2)
Other:
- note added: "i2c-display\n"
- note added: "i2c-ext\n"
- note removed: "i2c-a"
Changed lines of the file:
@@
 $EndComp
 Text Notes 2050 6500 0    60   ~ 0
-i2c-a
+i2c-display\n
 $Comp
 L hog32a-rescue:+3V3 #PWR017
@@
 $EndComp
 Wire Wire Line
-	5050 4250 4850 4250
+	5050 4250 4950 4250
 $Comp
 L Connector:Conn_01x02_Female J8
@@
 	0    1    1    0
 $EndComp
+$Comp
+L Connector:Conn_01x02_Male J16
+U 1 1 5CE314F3
+P 4500 3100
+F 0 "J16" H 4606 3278 50  0000 C CNN
+F 1 "Conn_01x02_Male" H 4100 3050 50  0000 C CNN
+F 2 "Connector_PinHeader_2.54mm:PinHeader_1x02_P2.54mm_Vertical" H 4500 3100 50  0001 C CNN
+F 3 "~" H 4500 3100 50  0001 C CNN
+	1    4500 3100
+	1    0    0    -1
+$EndComp
+Text GLabel 4700 2850 0    60   Input ~ 0
+RESET
+Wire Wire Line
+	4700 3100 4700 2850
+Wire Wire Line
+	4950 3750 4700 3750
+Wire Wire Line
+	4700 3750 4700 3200
+Wire Wire Line
+	4950 3750 4950 4250
+Connection ~ 4950 4250
+Wire Wire Line
+	4950 4250 4850 4250
+$Comp
+L Connector:Screw_Terminal_01x04 J19
+U 1 1 5CE40CFD
+P 3350 5900
+F 0 "J19" H 3430 5892 50  0000 L CNN
+F 1 "Screw_Terminal_01x04" H 3430 5801 50  0000 L CNN
+F 2 "TerminalBlock_Phoenix:TerminalBlock_Phoenix_PT-1,5-4-3.5-H_1x04_P3.50mm_Horizontal" H 3350 5900 50  0001 C CNN
+F 3 "~" H 3350 5900 50  0001 C CNN
+	1    3350 5900
+	1    0    0    -1
+$EndComp
+Text GLabel 3150 5800 0    60   Input ~ 0
+2:SDA
+Text GLabel 3150 5900 0    60   Input ~ 0
+14:SCL
+$Comp
+L hog32a-rescue:GND #PWR0107
+U 1 1 5CE40FA5
+P 3000 6200
+F 0 "#PWR0107" H 3000 5950 50  0001 C CNN
+F 1 "GND" H 3000 6050 50  0000 C CNN
+F 2 "" H 3000 6200 50  0001 C CNN
+F 3 "" H 3000 6200 50  0001 C CNN
+	1    3000 6200
+	1    0    0    -1
+$EndComp
+$Comp
+L hog32a-rescue:+3V3 #PWR0108
+U 1 1 5CE41008
+P 2600 6100
+F 0 "#PWR0108" H 2600 5950 50  0001 C CNN
+F 1 "+3V3" H 2600 6240 50  0000 C CNN
+F 2 "" H 2600 6100 50  0001 C CNN
+F 3 "" H 2600 6100 50  0001 C CNN
+	1    2600 6100
+	1    0    0    -1
+$EndComp
+Wire Wire Line
+	3150 6000 3000 6000
+Wire Wire Line
+	3000 6000 3000 6200
+Wire Wire Line
+	2600 6100 3150 6100
+Text Notes 3050 5600 0    60   ~ 0
+i2c-ext\n
 $EndSCHEMATC
