File: hog32a.sch (KiCad schematic (older format))
At the start: 44 parts, among them J1 REG:3V3, J10 Conn_01x07, J11 Conn_01x06_Male, J12 dht22, J13 Screw_Terminal_01x02, J14 Conn_01x09_Female, J15 Conn_01x05, J16 Conn_01x02_Male, J17 Conn_01x12_Female, J18 Barrel_Jack_Switch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

Commit message: update
Parts:
- removed J17: Conn_01x12_Female, Connector_PinHeader_2.54mm:PinHeader_1x12_P2.54mm_Vertical, symbol Connector:Conn_01x12_Female
- added J?: Conn_01x11_Female, symbol Connector:Conn_01x11_Female
- C1, C2, C5, C6: footprint Capacitor_THT:CP_Radial_D4.0mm_P1.50mm -> Capacitor_THT:CP_Radial_D5.0mm_P2.50mm
- C3, C4: renamed from C?; footprint Capacitor_THT:CP_Radial_D4.0mm_P1.50mm -> Capacitor_THT:CP_Radial_D5.0mm_P2.50mm
Connections:
- net +3V3: now also J?.10 (Pin_10)
- net 0: now also J?.6 (Pin_6)
- net 14:SCL: now also J?.7 (Pin_7)
- net 18:DHT22: now also J?.4 (Pin_4)
- net 19: now also J?.3 (Pin_3)
- net 21: now also J?.2 (Pin_2)
- net 23: now also J?.1 (Pin_1)
- net 2:SDA: now also J?.8 (Pin_8)
- net 5:onewire: now also J?.5 (Pin_5)
- net GND: now also J?.9 (Pin_9)
- net VIN: no longer J14.9 (Pin_9), J15.2 (Pin_2)
- net V_SWITCH: now also J14.9 (Pin_9), J15.2 (Pin_2), J?.11 (Pin_11)
Changed lines of the file:
@@
 	1    0    0    -1
 $EndComp
-Text GLabel 3000 6800 0    60   Input ~ 0
-VIN
 Text GLabel 7250 5050 0    60   Input ~ 0
 26
@@
 Text GLabel 10600 2050 0    60   Input ~ 0
 0
-Text GLabel 10600 2650 0    60   Input ~ 0
-VIN
-$Comp
-L hog32a-rescue:+5V #PWR036
-U 1 1 5B927367
-P 10150 2550
-F 0 "#PWR036" H 10150 2400 50  0001 C CNN
-F 1 "+5V" H 10150 2690 50  0000 C CNN
-F 2 "" H 10150 2550 50  0001 C CNN
-F 3 "" H 10150 2550 50  0001 C CNN
-	1    10150 2550
-	1    0    0    -1
-$EndComp
 Text GLabel 9100 1300 2    60   Input ~ 0
 22
@@
 	1    0    0    -1
 $EndComp
-Wire Wire Line
-	10600 2550 10150 2550
 Wire Wire Line
 	1150 3450 750  3450
@@
 	1    0    0    -1
 $EndComp
-Text GLabel 6200 2500 0    60   Input ~ 0
-VIN
 $Comp
 L hog32a-rescue:+5V #PWR0105
@@
 Wire Wire Line
 	10600 2350 9850 2350
-$Comp
-L Connector:Conn_01x12_Female J17
-U 1 1 5CEA2EDB
-P 10800 2050
-F 0 "J17" H 10827 2026 50  0000 L CNN
-F 1 "Conn_01x12_Female" V 10950 1700 50  0000 L CNN
-F 2 "Connector_PinHeader_2.54mm:PinHeader_1x12_P2.54mm_Vertical" H 10800 2050 50  0001 C CNN
-F 3 "~" H 10800 2050 50  0001 C CNN
-	1    10800 2050
-	1    0    0    -1
-$EndComp
 $Comp
 L Connector:Conn_01x09_Female J14
@@
 F 0 "C2" H 1232 2304 50  0000 R CNN
 F 1 "22uF" H 1232 2395 50  0000 R CNN
-F 2 "Capacitor_THT:CP_Radial_D4.0mm_P1.50mm" H 1388 2200 50  0001 C CNN
+F 2 "Capacitor_THT:CP_Radial_D5.0mm_P2.50mm" H 1388 2200 50  0001 C CNN
 F 3 "~" H 1350 2350 50  0001 C CNN
 	1    1350 2350
@@
 F 0 "C1" H 1468 2096 50  0000 L CNN
 F 1 "10uF" H 1468 2005 50  0000 L CNN
-F 2 "Capacitor_THT:CP_Radial_D4.0mm_P1.50mm" H 1388 1900 50  0001 C CNN
+F 2 "Capacitor_THT:CP_Radial_D5.0mm_P2.50mm" H 1388 1900 50  0001 C CNN
 F 3 "~" H 1350 2050 50  0001 C CNN
 	1    1350 2050
@@
 F 0 "C6" H 1232 3454 50  0000 R CNN
 F 1 "22uF" H 1232 3545 50  0000 R CNN
-F 2 "Capacitor_THT:CP_Radial_D4.0mm_P1.50mm" H 1388 3350 50  0001 C CNN
+F 2 "Capacitor_THT:CP_Radial_D5.0mm_P2.50mm" H 1388 3350 50  0001 C CNN
 F 3 "~" H 1350 3500 50  0001 C CNN
 	1    1350 3500
@@
 F 0 "C5" H 1468 3246 50  0000 L CNN
 F 1 "10uF" H 1468 3155 50  0000 L CNN
-F 2 "Capacitor_THT:CP_Radial_D4.0mm_P1.50mm" H 1388 3050 50  0001 C CNN
+F 2 "Capacitor_THT:CP_Radial_D5.0mm_P2.50mm" H 1388 3050 50  0001 C CNN
 F 3 "~" H 1350 3200 50  0001 C CNN
 	1    1350 3200
@@
 	1350 3050 2250 3050
 $Comp
-L Device:CP C?
+L Device:CP C3
 U 1 1 5CE56B2E
 P 1250 5500
-F 0 "C?" H 1368 5546 50  0000 L CNN
+F 0 "C3" H 1368 5546 50  0000 L CNN
 F 1 "1uF" H 1368 5455 50  0000 L CNN
-F 2 "Capacitor_THT:CP_Radial_D4.0mm_P1.50mm" H 1288 5350 50  0001 C CNN
+F 2 "Capacitor_THT:CP_Radial_D5.0mm_P2.50mm" H 1288 5350 50  0001 C CNN
 F 3 "~" H 1250 5500 50  0001 C CNN
 	1    1250 5500
@@
 $EndComp
 $Comp
-L Device:CP C?
+L Device:CP C4
 U 1 1 5CE57007
 P 2200 5500
-F 0 "C?" H 2318 5546 50  0000 L CNN
+F 0 "C4" H 2318 5546 50  0000 L CNN
 F 1 "1uF" H 2318 5455 50  0000 L CNN
-F 2 "Capacitor_THT:CP_Radial_D4.0mm_P1.50mm" H 2238 5350 50  0001 C CNN
+F 2 "Capacitor_THT:CP_Radial_D5.0mm_P2.50mm" H 2238 5350 50  0001 C CNN
 F 3 "~" H 2200 5500 50  0001 C CNN
 	1    2200 5500
 	1    0    0    -1
 $EndComp
+Text GLabel 3000 6800 0    60   Input ~ 0
+V_SWITCH
+Text GLabel 6200 2500 0    60   Input ~ 0
+V_SWITCH
+Text GLabel 10600 2550 0    60   Input ~ 0
+V_SWITCH
+$Comp
+L Connector:Conn_01x11_Female J?
+U 1 1 5CE6122B
+P 10800 2050
+F 0 "J?" H 10827 2076 50  0000 L CNN
+F 1 "Conn_01x11_Female" H 10827 1985 50  0000 L CNN
+F 2 "" H 10800 2050 50  0001 C CNN
+F 3 "~" H 10800 2050 50  0001 C CNN
+	1    10800 2050
+	1    0    0    -1
+$EndComp

Commit message: update
Parts:
- J17: renamed from J?; footprint (none) -> Connector_PinHeader_2.54mm:PinHeader_1x11_P2.54mm_Vertical
Connections:
- net +3V3: now also J5.3 (Pin_3); no longer J5.4 (Pin_4)
- net GND: now also J5.4 (Pin_4); no longer J5.3 (Pin_3)
Changed lines of the file:
@@
 L hog32a-rescue:GND #PWR015
 U 1 1 5B88CAD4
-P 2100 6900
-F 0 "#PWR015" H 2100 6650 50  0001 C CNN
-F 1 "GND" H 2100 6750 50  0000 C CNN
-F 2 "" H 2100 6900 50  0001 C CNN
-F 3 "" H 2100 6900 50  0001 C CNN
-	1    2100 6900
+P 2250 7000
+F 0 "#PWR015" H 2250 6750 50  0001 C CNN
+F 1 "GND" H 2250 6850 50  0000 C CNN
+F 2 "" H 2250 7000 50  0001 C CNN
+F 3 "" H 2250 7000 50  0001 C CNN
+	1    2250 7000
 	1    0    0    -1
 $EndComp
@@
 L hog32a-rescue:+3V3 #PWR016
 U 1 1 5B88CCC7
-P 1800 7150
-F 0 "#PWR016" H 1800 7000 50  0001 C CNN
-F 1 "+3V3" H 1800 7290 50  0000 C CNN
-F 2 "" H 1800 7150 50  0001 C CNN
-F 3 "" H 1800 7150 50  0001 C CNN
-	1    1800 7150
+P 1750 6900
+F 0 "#PWR016" H 1750 6750 50  0001 C CNN
+F 1 "+3V3" H 1750 7040 50  0000 C CNN
+F 2 "" H 1750 6900 50  0001 C CNN
+F 3 "" H 1750 6900 50  0001 C CNN
+	1    1750 6900
 	1    0    0    -1
 $EndComp
@@
 Wire Wire Line
 	1150 2100 750  2100
-Wire Wire Line
-	1800 7150 2250 7150
-Wire Wire Line
-	2250 7150 2250 7000
-Wire Wire Line
-	2250 6900 2100 6900
 Connection ~ 5800 7100
 Wire Wire Line
@@
 V_SWITCH
 $Comp
-L Connector:Conn_01x11_Female J?
+L Connector:Conn_01x11_Female J17
 U 1 1 5CE6122B
 P 10800 2050
-F 0 "J?" H 10827 2076 50  0000 L CNN
+F 0 "J17" H 10827 2076 50  0000 L CNN
 F 1 "Conn_01x11_Female" H 10827 1985 50  0000 L CNN
-F 2 "" H 10800 2050 50  0001 C CNN
+F 2 "Connector_PinHeader_2.54mm:PinHeader_1x11_P2.54mm_Vertical" H 10800 2050 50  0001 C CNN
 F 3 "~" H 10800 2050 50  0001 C CNN
 	1    10800 2050
 	1    0    0    -1
 $EndComp
+Wire Wire Line
+	2250 6900 1750 6900
 $EndSCHEMATC

Commit message: update
Parts:
- removed J17: Conn_01x11_Female, Connector_PinHeader_2.54mm:PinHeader_1x11_P2.54mm_Vertical, symbol Connector:Conn_01x11_Female
- added J17: Conn_01x10_Female, Connector_PinSocket_2.54mm:PinSocket_1x10_P2.54mm_Vertical, symbol Connector:Conn_01x10_Female
- added R10, R9: R, Resistor_THT:R_Axial_DIN0204_L3.6mm_D1.6mm_P1.90mm_Vertical, symbol Device:R
- J10: footprint Pin_Headers:Pin_Header_Straight_1x07_Pitch2.54mm -> Connector_PinHeader_2.54mm:PinHeader_1x07_P2.54mm_Vertical
- J14: footprint Connector_PinHeader_2.54mm:PinHeader_1x09_P2.54mm_Vertical -> Connector_PinSocket_2.54mm:PinSocket_1x09_P2.54mm_Vertical
- J8: footprint Connector_PinHeader_2.54mm:PinHeader_1x02_P2.54mm_Vertical -> Connector_PinSocket_2.54mm:PinSocket_1x02_P2.54mm_Vertical
Connections:
- net +3V3: now also J17.9 (Pin_9)
- net 0: now also J17.5 (Pin_5)
- net 14:SCL: now also J17.6 (Pin_6)
- net 18:DHT22: now also J17.3 (Pin_3)
- net 19: now also J17.2 (Pin_2)
- net 21: now also J17.1 (Pin_1)
- net 23: now also J14.2 (Pin_2)
- net 2:SDA: now also J17.7 (Pin_7)
- net 34: now also R10.1, R9.2; no longer J14.2 (Pin_2)
- net 5:onewire: now also J17.4 (Pin_4)
- net GND: now also J17.8 (Pin_8), R10.2
- net V_SWITCH: now also J17.10 (Pin_10), R9.1
Changed lines of the file:
@@
 	1    0    0    -1
 $EndComp
-Text GLabel 10600 1550 0    60   Input ~ 0
-23
 $Comp
 L hog32a-rescue:+3V3 #PWR032
@@
 Text GLabel 10800 5050 1    60   Input ~ 0
 DIO5
-Text GLabel 6200 1800 0    60   Input ~ 0
+Text GLabel 5700 1150 2    60   Input ~ 0
 34
 Text GLabel 6200 2000 0    60   Input ~ 0
@@
 F 0 "J10" H 9700 5700 50  0000 C CNN
 F 1 "Conn_01x07" H 9700 4900 50  0000 C CNN
-F 2 "Pin_Headers:Pin_Header_Straight_1x07_Pitch2.54mm" H 9700 5300 50  0001 C CNN
+F 2 "Connector_PinHeader_2.54mm:PinHeader_1x07_P2.54mm_Vertical" H 9700 5300 50  0001 C CNN
 F 3 "" H 9700 5300 50  0001 C CNN
 	1    9700 5300
@@
 F 0 "J8" H 3250 4250 50  0000 C CNN
 F 1 "Conn_01x02_Female" H 3300 4450 50  0000 C CNN
-F 2 "Connector_PinHeader_2.54mm:PinHeader_1x02_P2.54mm_Vertical" H 3150 4350 50  0001 C CNN
+F 2 "Connector_PinSocket_2.54mm:PinSocket_1x02_P2.54mm_Vertical" H 3150 4350 50  0001 C CNN
 F 3 "~" H 3150 4350 50  0001 C CNN
 	1    3150 4350
@@
 Wire Wire Line
 	10600 2350 9850 2350
-$Comp
-L Connector:Conn_01x09_Female J14
-U 1 1 5CEA3175
-P 6400 2100
-F 0 "J14" H 6427 2126 50  0000 L CNN
-F 1 "Conn_01x09_Female" V 6600 1800 50  0000 L CNN
-F 2 "Connector_PinHeader_2.54mm:PinHeader_1x09_P2.54mm_Vertical" H 6400 2100 50  0001 C CNN
-F 3 "~" H 6400 2100 50  0001 C CNN
-	1    6400 2100
-	1    0    0    -1
-$EndComp
 Wire Wire Line
 	5250 3450 5250 2950
@@
 Text GLabel 10600 2550 0    60   Input ~ 0
 V_SWITCH
-$Comp
-L Connector:Conn_01x11_Female J17
-U 1 1 5CE6122B
+Wire Wire Line
+	2250 6900 1750 6900
+Text GLabel 6200 1800 0    60   Input ~ 0
+23
+$Comp
+L Connector:Conn_01x10_Female J17
+U 1 1 5CE5762D
 P 10800 2050
-F 0 "J17" H 10827 2076 50  0000 L CNN
-F 1 "Conn_01x11_Female" H 10827 1985 50  0000 L CNN
-F 2 "Connector_PinHeader_2.54mm:PinHeader_1x11_P2.54mm_Vertical" H 10800 2050 50  0001 C CNN
+F 0 "J17" H 10827 2026 50  0000 L CNN
+F 1 "Conn_01x10_Female" H 10827 1935 50  0000 L CNN
+F 2 "Connector_PinSocket_2.54mm:PinSocket_1x10_P2.54mm_Vertical" H 10800 2050 50  0001 C CNN
 F 3 "~" H 10800 2050 50  0001 C CNN
 	1    10800 2050
 	1    0    0    -1
 $EndComp
-Wire Wire Line
-	2250 6900 1750 6900
+$Comp
+L Device:R R9
+U 1 1 5CE5AADE
+P 5400 950
+F 0 "R9" H 5470 996 50  0000 L CNN
+F 1 "R" H 5470 905 50  0000 L CNN
+F 2 "Resistor_THT:R_Axial_DIN0204_L3.6mm_D1.6mm_P1.90mm_Vertical" V 5330 950 50  0001 C CNN
+F 3 "~" H 5400 950 50  0001 C CNN
+	1    5400 950
+	1    0    0    -1
+$EndComp
+$Comp
+L Device:R R10
+U 1 1 5CE6153A
+P 5400 1350
+F 0 "R10" H 5470 1396 50  0000 L CNN
+F 1 "R" H 5470 1305 50  0000 L CNN
+F 2 "Resistor_THT:R_Axial_DIN0204_L3.6mm_D1.6mm_P1.90mm_Vertical" V 5330 1350 50  0001 C CNN
+F 3 "~" H 5400 1350 50  0001 C CNN
+	1    5400 1350
+	1    0    0    -1
+$EndComp
+$Comp
+L hog32a-rescue:GND #PWR0109
+U 1 1 5CE6162F
+P 5400 1500
+F 0 "#PWR0109" H 5400 1250 50  0001 C CNN
+F 1 "GND" H 5405 1327 50  0000 C CNN
+F 2 "" H 5400 1500 50  0001 C CNN
+F 3 "" H 5400 1500 50  0001 C CNN
+	1    5400 1500
+	1    0    0    -1
+$EndComp
+Text GLabel 5400 700  0    60   Input ~ 0
+V_SWITCH
+Wire Wire Line
+	5400 800  5400 700
+Wire Wire Line
+	5400 1100 5400 1150
+Wire Wire Line
+	5400 1150 5700 1150
+Connection ~ 5400 1150
+Wire Wire Line
+	5400 1150 5400 1200
+$Comp
+L Connector:Conn_01x09_Female J14
+U 1 1 5CE770B3
+P 6400 2100
+F 0 "J14" H 6427 2126 50  0000 L CNN
+F 1 "Conn_01x09_Female" H 6427 2035 50  0000 L CNN
+F 2 "Connector_PinSocket_2.54mm:PinSocket_1x09_P2.54mm_Vertical" H 6400 2100 50  0001 C CNN
+F 3 "~" H 6400 2100 50  0001 C CNN
+	1    6400 2100
+	1    0    0    -1
+$EndComp
 $EndSCHEMATC

Commit message: update
Parts:
- J16, J2: footprint Connector_PinHeader_2.54mm:PinHeader_1x02_P2.54mm_Vertical -> Connector_PinSocket_2.54mm:PinSocket_1x02_P2.54mm_Vertical
- J4: footprint Pin_Headers:Pin_Header_Straight_1x07_Pitch2.54mm -> Connector_PinSocket_2.54mm:PinSocket_1x07_P2.54mm_Vertical
Changed lines of the file:
@@
 F 0 "J4" H 4650 7250 50  0000 C CNN
 F 1 "sdcard" H 4650 6450 50  0000 C CNN
-F 2 "Pin_Headers:Pin_Header_Straight_1x07_Pitch2.54mm" H 4650 6850 50  0001 C CNN
+F 2 "Connector_PinSocket_2.54mm:PinSocket_1x07_P2.54mm_Vertical" H 4650 6850 50  0001 C CNN
 F 3 "" H 4650 6850 50  0001 C CNN
 	1    4650 6850
@@
 F 0 "J2" H 2856 1978 50  0000 C CNN
 F 1 "Conn_01x02_Male" H 3350 1750 50  0000 C CNN
-F 2 "Connector_PinHeader_2.54mm:PinHeader_1x02_P2.54mm_Vertical" H 2750 1800 50  0001 C CNN
+F 2 "Connector_PinSocket_2.54mm:PinSocket_1x02_P2.54mm_Vertical" H 2750 1800 50  0001 C CNN
 F 3 "~" H 2750 1800 50  0001 C CNN
 	1    2750 1800
@@
 F 0 "J16" H 4606 3278 50  0000 C CNN
 F 1 "Conn_01x02_Male" H 4100 3050 50  0000 C CNN
-F 2 "Connector_PinHeader_2.54mm:PinHeader_1x02_P2.54mm_Vertical" H 4500 3100 50  0001 C CNN
+F 2 "Connector_PinSocket_2.54mm:PinSocket_1x02_P2.54mm_Vertical" H 4500 3100 50  0001 C CNN
 F 3 "~" H 4500 3100 50  0001 C CNN
 	1    4500 3100

Commit message: update
Parts:
- removed J14: Conn_01x09_Female, Connector_PinSocket_2.54mm:PinSocket_1x09_P2.54mm_Vertical, symbol Connector:Conn_01x09_Female
- added J14: Conn_01x10_Female, Connector_PinSocket_2.54mm:PinSocket_1x10_P2.54mm_Vertical, symbol Connector:Conn_01x10_Female
- added JP1: SolderJumper_2_Bridged, Jumper:SolderJumper-2_P1.3mm_Bridged_RoundedPad1.0x1.5mm, symbol Jumper:SolderJumper_2_Bridged
- added JP2: SolderJumper_2_Open, Jumper:SolderJumper-2_P1.3mm_Open_RoundedPad1.0x1.5mm, symbol Jumper:SolderJumper_2_Open
- J10: footprint Connector_PinHeader_2.54mm:PinHeader_1x07_P2.54mm_Vertical -> Connector_PinSocket_2.54mm:PinSocket_1x07_P2.54mm_Vertical
- J3: footprint Connector_PinHeader_2.54mm:PinHeader_1x06_P2.54mm_Vertical -> Connector_PinSocket_2.54mm:PinSocket_1x06_P2.54mm_Vertical
Connections:
- net +3V3: now also J14.8 (Pin_8)
- net +5V: now also J14.7 (Pin_7)
- net 12: now also J14.5 (Pin_5)
- net 13: now also J14.4 (Pin_4)
- net 23: now also J14.2 (Pin_2)
- net 35: now also J14.3 (Pin_3)
- net GND: now also J14.6 (Pin_6)
- net RESET: now also J14.1 (Pin_1)
- net VIN: now also J14.10 (Pin_10), JP2.2 (B)
- net V_SWITCH: now also J14.9 (Pin_9), JP2.1 (A)
- net at J16.2 (Pin_2), U3.5 (DRV): now also JP1.1 (A); no longer R2.2
- new net: JP1.2 (B), R2.2
Other:
- moved on the sheet: J15, J19, J3, Q1, Q2, R2, R3
