File: hog32a.kicad_pcb (KiCad board)
At the start: 2 copper layers, 51.6 x 75.9 mm, 38 parts, among them J1 REG:3V3, J10 Conn_01x07, J11 Conn_01x16, J12 dht22, J13 9602-a, J14 satx, J15 Conn_01x05, J16 LBO, J19 9602-b, J2 prog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

Commit message: update;
Parts:
- removed J16: LBO, Pin_Headers:Pin_Header_Straight_2x03_Pitch2.54mm
- removed J19: 9602-b, Pin_Headers:Pin_Header_Straight_1x08_Pitch2.54mm
- added BT1: Battery_Cell, Battery:BatteryHolder_Keystone_3000_1x12mm, F.Cu at (85.3, 74.4)
- added J17: Conn_01x12_Female, Connector_PinHeader_2.54mm:PinHeader_1x12_P2.54mm_Vertical, F.Cu at (121.9, 66.0)
- added J18: Barrel_Jack_Switch, Connector_BarrelJack:BarrelJack_Horizontal, F.Cu at (77.2, 95.5)
- added J8: Conn_01x02_Female, Connector_PinHeader_2.54mm:PinHeader_1x02_P2.54mm_Vertical, F.Cu at (94.0, 52.8)
- added S1: EG1218, digikey-footprints:Switch_Slide_11.6x4mm_EG1218, F.Cu at (115.3, 72.4)
- added U3: TPL5111, Package_TO_SOT_SMD:SOT-23-6_Handsoldering, F.Cu at (86.9, 61.0)
- J11: value Conn_01x16 -> Conn_01x06_Male; footprint Pin_Headers:Pin_Header_Straight_1x16_Pitch2.54mm -> Connector_PinHeader_2.54mm:PinHeader_1x06_P2.54mm_Vertical
- J13: value 9602-a -> Screw_Terminal_01x02; footprint Pin_Headers:Pin_Header_Straight_1x06_Pitch2.54mm -> TerminalBlock_Phoenix:TerminalBlock_Phoenix_PT-1,5-2-3.5-H_1x02_P3.50mm_Horizontal
- J14: value satx -> Conn_01x09_Female; footprint Pin_Headers:Pin_Header_Straight_1x04_Pitch2.54mm -> Connector_PinHeader_2.54mm:PinHeader_1x09_P2.54mm_Vertical
- J2: value prog -> Conn_01x02_Male; footprint Pin_Headers:Pin_Header_Straight_1x07_Pitch2.54mm -> Connector_PinHeader_2.54mm:PinHeader_1x02_P2.54mm_Vertical
- J3: value VINS -> Conn_01x06_Female; footprint TerminalBlocks_Phoenix:TerminalBlock_Phoenix_PT-3.5mm_2pol -> Connector_PinHeader_2.54mm:PinHeader_1x06_P2.54mm_Vertical
- Q1: footprint TO_SOT_Packages_THT:TO-92_Molded_Narrow -> Package_TO_SOT_THT:TO-92
- Q2: value Q_NPN_EBC -> Q_PNP_BCE; footprint TO_SOT_Packages_THT:TO-92_Molded_Narrow -> Package_TO_SOT_THT:TO-220-3_Vertical
- R2: value 10K -> 1K; footprint Resistors_THT:R_Axial_DIN0204_L3.6mm_D1.6mm_P1.90mm_Vertical -> Resistor_THT:R_Axial_DIN0204_L3.6mm_D1.6mm_P1.90mm_Vertical
- R3: value 10K -> 50 ohms; footprint Resistors_THT:R_Axial_DIN0204_L3.6mm_D1.6mm_P1.90mm_Vertical -> Resistor_THT:R_Axial_DIN0204_L3.6mm_D1.6mm_P1.90mm_Vertical
- moved J3 45.9 mm to (88.9, 55.6), turned to 270 degrees
- moved J11 45.8 mm to (113.5, 82.0)
- moved J13 42.0 mm to (98.3, 101.1)
- moved J2 34.3 mm to (80.3, 90.9), turned to 90 degrees
- moved Q2 26.7 mm to (74.7, 60.5), turned to 270 degrees
- moved J14 20.4 mm to (74.9, 70.9)
- moved Q1 19.2 mm to (80.5, 59.2), turned to 270 degrees
- moved C2 16.6 mm to (93.7, 95.5), turned to 180 degrees
- moved SW2 9.80 mm to (109.2, 75.7)
- moved D2 9.24 mm to (80.0, 86.4), turned to 0 degrees
- moved R2 8.90 mm to (87.4, 65.0), turned to 180 degrees
- moved SW1 8.72 mm to (111.5, 63.2)
- moved C3 8.66 mm to (95.5, 73.7)
- moved R8 8.39 mm to (113.0, 76.2)
- moved R3 7.62 mm to (81.5, 65.3), turned to 180 degrees
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Connections:
- D2 pad 2: VIN -> V_SWITCH
- J11 pad 1: RESET -> (no net)
- J11 pad 2: 35 -> TX0
- J11 pad 3: 23:SAT_SLEEP -> RX0
- J11 pad 4: 22 -> VBUS
- J11 pad 5: 21 -> (no net)
- J11 pad 6: 19 -> GND
- J13 pad 1: (no net) -> GND
- J13 pad 2: 34 -> VIN
- J14 pad 1: SAT_RING_INDICATOR -> RESET
- J14 pad 2: SAT_NETWORK_AVAIL -> 34
- J14 pad 3: 23:SAT_SLEEP -> 35
- J14 pad 4: SAT_LION -> 13
- J2 pad 1: GND -> V_SWITCH
- J2 pad 2: (no net) -> VIN
- J3 pad 1: GND -> DIO5
- J3 pad 2: VIN -> 27
- Q1 pad 1: DTR -> GND
- Q1 pad 3: 0 -> Net-(Q1-Pad3)
- Q2 pad 1: RTS -> Net-(Q2-Pad1)
- Q2 pad 2: Net-(Q2-Pad2) -> V_SWITCH
- Q2 pad 3: RESET -> VIN
- R2 pad 2: RTS -> Net-(R2-Pad2)
- R3 pad 1: Net-(Q2-Pad2) -> Net-(Q2-Pad1)
- R3 pad 2: DTR -> Net-(Q1-Pad3)
- U1 pad 37: 23:SAT_SLEEP -> 23
Routing:
- net 23:SAT_SLEEP: track 92.7 -> 0.00 mm, vias 4 -> 0
- net GND: track 330.6 -> 238.1 mm, vias 9 -> 8
- net 17: track 78.4 -> 0.00 mm, vias 1 -> 0
- net 4: track 78.2 -> 0.00 mm, vias 1 -> 0
- net 16: track 75.9 -> 0.00 mm, vias 1 -> 0
- net 15: track 73.3 -> 0.00 mm, vias 1 -> 0
- net +5V: track 91.9 -> 21.2 mm, vias 3 -> 0
- net VIN: track 87.8 -> 26.3 mm, vias 5 -> 2
- net 13: track 55.5 -> 0.00 mm, vias 1 -> 0
- net RESET: track 93.5 -> 44.7 mm
- net TX0: track 47.7 -> 0.00 mm, vias 5 -> 0
- net +3V3: track 202.1 -> 163.8 mm, vias 7 -> 3
- net 34: track 37.0 -> 0.00 mm, vias 1 -> 0
- net DTR: track 35.4 -> 0.00 mm, vias 1 -> 0
- net RTS: track 34.3 -> 0.00 mm
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Other:
- outline, holes or cut-outs redrawn
- board text removed: "13"
- board text removed: "34"

Commit message: update
Parts:
- added J16: Conn_01x02_Male, Connector_PinHeader_2.54mm:PinHeader_1x02_P2.54mm_Vertical, F.Cu at (23.4, 36.2)
- added J19: Screw_Terminal_01x04, TerminalBlock_Phoenix:TerminalBlock_Phoenix_PT-1,5-4-3.5-H_1x04_P3.50mm_Horizontal, F.Cu at (51.9, 49.3)
- moved J17 92.7 mm to (55.1, 1.82), turned to 0 degrees
- moved R7 88.2 mm to (37.3, 22.8)
- moved C6 82.1 mm to (28.2, 64.6)
- moved R3 81.2 mm to (6.64, 33.9), turned to 0 degrees
- moved C5 81.1 mm to (31.8, 64.6)
- moved R2 80.9 mm to (13.0, 33.1), turned to 0 degrees
- moved J11 80.7 mm to (39.4, 50.1)
- moved U3 79.6 mm to (13.7, 29.6)
- moved J10 79.4 mm to (1.90, 1.81)
- moved J12 79.4 mm to (41.2, 28.4)
- moved J14 79.4 mm to (1.81, 40.0)
- moved J3 79.4 mm to (15.8, 24.7)
- moved J4 79.4 mm to (32.5, 60.6)
- moved J5 79.4 mm to (27.2, 29.4)
- moved J7 79.4 mm to (19.0, 5.95)
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Routing:
- net GND: track 238.1 -> 60.3 mm, vias 8 -> 2
- net +3V3: track 163.8 -> 15.1 mm, vias 3 -> 0
- net 5:onewire: track 53.9 -> 0.00 mm
- net RESET: track 44.7 -> 0.00 mm, vias 4 -> 0
- net 14:SCL: track 48.4 -> 5.17 mm, vias 1 -> 0
- net 21: track 43.7 -> 0.75 mm, vias 3 -> 0
- net 0: track 36.8 -> 0.00 mm, vias 3 -> 0
- net 32: track 31.6 -> 0.00 mm
- net 12: track 31.2 -> 0.00 mm, vias 7 -> 0
- net 19: track 30.0 -> 0.00 mm, vias 1 -> 0
- net 33: track 29.4 -> 0.27 mm
- net 25: track 26.3 -> 0.75 mm
- net 18:DHT22: track 25.4 -> 0.00 mm, vias 1 -> 0
- net 2:SDA: track 28.4 -> 4.33 mm, vias 1 -> 0
- net Net-(C1-Pad1): track 48.7 -> 26.0 mm
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Other:
- board size 51.6 x 75.9 mm -> 57.1 x 87.6 mm

Commit message: update
Parts:
- C1, C5: value 10 uF -> 10uF; footprint Capacitors_THT:C_Disc_D3.0mm_W1.6mm_P2.50mm -> Capacitor_THT:CP_Radial_D5.0mm_P2.50mm
- C2, C6: value 22 uF -> 22uF; footprint Capacitors_THT:C_Disc_D3.0mm_W1.6mm_P2.50mm -> Capacitor_THT:CP_Radial_D5.0mm_P2.50mm
- C3, C4: footprint Capacitors_THT:C_Disc_D3.0mm_W1.6mm_P2.50mm -> Capacitor_THT:CP_Radial_D5.0mm_P2.50mm
- moved U1 39.2 mm to (42.4, 13.5)
- moved C3 20.8 mm to (45.6, 50.3), turned to 180 degrees
- moved C4 18.7 mm to (36.5, 50.3), turned to 0 degrees
- moved R7 15.5 mm to (51.8, 28.5)
- moved SW1 14.0 mm to (43.1, 45.5), turned to 90 degrees
- moved J8 13.7 mm to (14.0, 33.8), turned to 90 degrees
- moved C5 11.1 mm to (41.3, 70.3), turned to 180 degrees
- moved J11 11.0 mm to (46.0, 58.9)
- moved C2 10.4 mm to (13.5, 70.1), turned to 0 degrees
- moved R8 10.3 mm to (44.4, 54.6)
- moved C1 9.62 mm to (21.9, 70.2), turned to 180 degrees
- moved R1 9.43 mm to (43.5, 33.8), turned to 270 degrees
- moved R4 9.09 mm to (39.6, 33.8), turned to 270 degrees
- moved R3 7.96 mm to (1.39, 27.9)
- moved D2 7.42 mm to (24.6, 57.4), turned to 180 degrees
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Connections:
- C2 pad 1: GND -> +3V3
- C2 pad 2: +3V3 -> GND
- C6 pad 1: GND -> +5V
- C6 pad 2: +5V -> GND
Routing:
- net GND: track 60.3 -> 208.3 mm, vias 2 -> 0
- net +3V3: track 15.1 -> 68.1 mm
- net VIN: track 6.06 -> 51.5 mm, vias 2 -> 0
- net Net-(C1-Pad1): track 26.0 -> 7.01 mm, vias 1 -> 0
- net 0: track 0.00 -> 18.0 mm
- net RESET: track 0.00 -> 6.50 mm
- net 14:SCL: track 5.17 -> 0.00 mm
- net Net-(Q1-Pad3): track 0.00 -> 4.85 mm
- net DIO5: track 0.00 -> 4.37 mm
- net 2:SDA: track 4.33 -> 0.00 mm
- net Net-(Q2-Pad1): track 0.00 -> 4.27 mm
- net 27: track 0.79 -> 4.94 mm
- net Net-(Q1-Pad2): track 0.00 -> 3.98 mm
- net 26: track 0.89 -> 4.81 mm
- net 32: track 0.00 -> 3.86 mm
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Other:
- board size 57.1 x 87.6 mm -> 58 x 82 mm
- rule trace_min: 0.2 -> 0.1524
- rule via_min_drill: 0.3 -> 0.254
- rule via_min_size: 0.4 -> 0.508

Commit message: update
Parts:
- J17: value Conn_01x12_Female -> Conn_01x11_Female; footprint Connector_PinHeader_2.54mm:PinHeader_1x12_P2.54mm_Vertical -> Connector_PinHeader_2.54mm:PinHeader_1x11_P2.54mm_Vertical
- moved S1 47.1 mm to (2.33, 32.9), turned to 270 degrees
- moved J8 13.7 mm to (1.94, 27.2)
- moved R2 9.36 mm to (16.3, 33.0)
- moved Q2 5.72 mm to (7.26, 32.4)
- moved R3 3.95 mm to (5.34, 27.8)
- moved J2 3.72 mm to (12.0, 62.1), turned to 0 degrees
- moved R8 3.59 mm to (47.9, 53.7), turned to 270 degrees
- moved U3 2.18 mm to (17.5, 29.6)
- moved BT1 1.72 mm to (14.5, 48.1)
- moved J16 1.37 mm to (29.1, 37.1)
- moved J3 0.99 mm to (15.0, 24.1)
- moved J14 0.78 mm to (1.76, 43.3)
- moved D1 0.72 mm to (30.7, 58.0)
- moved D2 0.68 mm to (24.5, 58.0)
- moved J4 0.58 mm to (34.2, 63.9)
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Connections:
- J14 pad 9: VIN -> V_SWITCH
- J15 pad 2: VIN -> V_SWITCH
- J17 pad 11: +5V -> V_SWITCH
Routing:
- net V_SWITCH: track 0.00 -> 141.7 mm
- net +3V3: track 68.1 -> 176.4 mm, vias 0 -> 1
- net +5V: track 0.00 -> 70.2 mm, vias 0 -> 2
- net GND: track 208.3 -> 274.2 mm
- net VIN: track 51.5 -> 30.8 mm
- net VBUS: track 0.00 -> 15.2 mm
- net Net-(Q1-Pad3): track 4.85 -> 0.00 mm
- net Net-(Q2-Pad1): track 4.27 -> 0.00 mm
- net Net-(Q1-Pad2): track 3.98 -> 0.00 mm
- net DIO3: track 5.52 -> 4.27 mm

Commit message: update
Parts:
- moved C2 33.2 mm to (46.7, 72.1), turned to 270 degrees
- moved C1 26.1 mm to (46.8, 77.8), turned to 270 degrees
- moved J13 21.9 mm to (2.79, 76.7)
- moved J1 21.1 mm to (40.0, 76.8)
- moved C4 14.1 mm to (28.6, 38.6)
- moved C3 12.9 mm to (33.7, 45.2)
- moved J6 11.8 mm to (27.6, 76.9)
- moved R8 11.1 mm to (48.5, 64.8)
- moved C6 10.3 mm to (22.6, 72.8), turned to 90 degrees
- moved J2 10.2 mm to (6.58, 70.8), turned to 180 degrees
- moved R1 9.89 mm to (35.9, 40.2)
- moved J12 9.53 mm to (56.2, 33.2)
- moved J18 9.01 mm to (14.0, 67.8)
- moved D2 8.48 mm to (31.3, 53.0), turned to 270 degrees
- moved D1 7.97 mm to (36.9, 53.0), turned to 270 degrees
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Connections:
- J5 pad 3: GND -> +3V3
- J5 pad 4: +3V3 -> GND
Routing:
- net GND: track 274.2 -> 88.3 mm
- net V_SWITCH: track 141.7 -> 3.22 mm
- net +3V3: track 176.4 -> 40.3 mm, vias 1 -> 0
- net +5V: track 70.2 -> 0.00 mm, vias 2 -> 0
- net VIN: track 30.8 -> 0.00 mm
- net 0: track 18.0 -> 0.00 mm
- net VBUS: track 15.2 -> 0.00 mm
- net Net-(C1-Pad1): track 7.01 -> 0.45 mm
- net 14:SCL: track 0.00 -> 4.02 mm
- net 2:SDA: track 0.00 -> 3.28 mm
- net Net-(BT1-Pad1): track 0.00 -> 2.35 mm
Other:
- outline, holes or cut-outs redrawn

Commit message: update
Parts:
- moved R7 28.4 mm to (80.7, 27.8)
- moved J12 26.4 mm to (82.6, 32.9)
- moved SW1 7.45 mm to (47.2, 36.0)
- moved SW2 6.29 mm to (40.5, 40.3)
- moved J4 2.17 mm to (38.0, 65.5)
Routing:
- net GND: track 88.3 -> 44.2 mm
- net RESET: track 6.50 -> 0.00 mm

Commit message: update
Parts:
- moved J12 63.5 mm to (20.3, 20.5), turned to 180 degrees
- moved R7 61.3 mm to (23.8, 5.28), turned to 270 degrees
- moved J16 21.8 mm to (40.6, 47.4)
- moved C6 17.3 mm to (7.78, 63.8)
- moved C5 13.4 mm to (22.6, 67.8)
- moved C3 12.2 mm to (45.7, 47.7), turned to 270 degrees
- moved R1 11.9 mm to (46.3, 34.4), turned to 90 degrees
- moved C2 11.7 mm to (35.8, 67.7)
- moved R8 9.23 mm to (48.7, 55.6)
- moved SW1 8.83 mm to (56.0, 35.6)
- moved J4 8.57 mm to (30.3, 61.8)
- moved C4 6.54 mm to (32.9, 43.6), turned to 270 degrees
- moved R4 6.29 mm to (37.6, 40.8)
- moved D2 5.43 mm to (36.6, 53.8)
- moved D1 4.75 mm to (32.5, 50.9)
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
Commit message: update
Parts:
- moved J11 0.46 mm to (43.5, 58.3)
Changed lines of the file:
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@@
   )
   (module Connector_PinHeader_2.54mm:PinHeader_1x06_P2.54mm_Vertical (layer F.Cu)
-    (at 43.625 57.85)
+    (at 43.525 58.3)
     (descr "Through hole straight pin header, 1x06, 2.54mm pitch, single row")
     (tags "Through hole pin header THT 1x06 2.54mm single row")
@@
   (gr_line (start 19.29 74.571) (end 30.89 74.571) (angle 90) (layer Dwgs.User) (width 0.2))
   (gr_line (start 29 0) (end 29 10.25) (layer Dwgs.User) (width 0.2))
-  (gr_text GND (at 42.995 66.81 90) (layer F.SilkS)
-    (effects (font (size 0.8 0.8) (thickness 0.2)))
-  )
-  (gr_line (start 43.28524 72.74768) (end 43.28524 72.7426) (angle 90) (layer F.SilkS) (width 0.2))
-  (gr_line (start 44.26 65.585) (end 47.308 65.585) (angle 90) (layer F.SilkS) (width 0.2))
+  (gr_text GND (at 42.895 67.26 90) (layer F.SilkS)
+    (effects (font (size 0.8 0.8) (thickness 0.2)))
+  )
+  (gr_line (start 43.18524 73.19768) (end 43.18524 73.1926) (angle 90) (layer F.SilkS) (width 0.2))
+  (gr_line (start 44.16 66.035) (end 47.208 66.035) (angle 90) (layer F.SilkS) (width 0.2))
   (gr_line (start 47.05664 54.66104) (end 44.23724 54.66104) (angle 90) (layer F.SilkS) (width 0.2))
-  (gr_text RTS (at 45.88824 56.24092 90) (layer F.SilkS)
-    (effects (font (size 0.8 0.8) (thickness 0.2)))
-  )
-  (gr_text TX (at 45.91872 58.5066 90) (layer F.SilkS)
-    (effects (font (size 0.8 0.8) (thickness 0.2)))
-  )
-  (gr_text VBS (at 45.99492 63.42912 90) (layer F.SilkS)
-    (effects (font (size 0.8 0.8) (thickness 0.2)))
-  )
-  (gr_text RX (at 45.90348 60.89928 90) (layer F.SilkS)
+  (gr_text RTS (at 45.78824 56.69092 90) (layer F.SilkS)
+    (effects (font (size 0.8 0.8) (thickness 0.2)))
+  )
+  (gr_text TX (at 45.81872 58.9566 90) (layer F.SilkS)
+    (effects (font (size 0.8 0.8) (thickness 0.2)))
+  )
+  (gr_text VBS (at 45.89492 63.87912 90) (layer F.SilkS)
+    (effects (font (size 0.8 0.8) (thickness 0.2)))
+  )
+  (gr_text RX (at 45.80348 61.34928 90) (layer F.SilkS)
     (effects (font (size 0.8 0.8) (thickness 0.2)))
   )
@@
     (effects (font (size 1.5 1.5) (thickness 0.25)) (justify mirror))
   )
-  (gr_text QUAHOG (at 27.05 14.95 90) (layer F.SilkS)
+  (gr_text QUAHOG (at 29.15 14.675 90) (layer F.SilkS)
     (effects (font (size 2.8 3) (thickness 0.3)))
   )
