File: hog32a.kicad_pcb (KiCad board)
At the start: 2 copper layers, 58 x 82 mm, 44 parts, among them J1 REG:3V3, J10 Conn_01x07, J11 Conn_01x06_Male, J12 dht22, J13 Screw_Terminal_01x02, J14 Conn_01x09_Female, J15 Conn_01x05, J16 Conn_01x02_Male, J17 Conn_01x11_Female, J18 Barrel_Jack_Switch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

Commit message: update
Parts:
- added R10: R, Resistor_THT:R_Axial_DIN0204_L3.6mm_D1.6mm_P1.90mm_Vertical, F.Cu at (14.0, 36.1)
- added R9: R, Resistor_THT:R_Axial_DIN0204_L3.6mm_D1.6mm_P1.90mm_Vertical, F.Cu at (12.2, 38.4)
- J14: footprint Connector_PinHeader_2.54mm:PinHeader_1x09_P2.54mm_Vertical -> Connector_PinSocket_2.54mm:PinSocket_1x09_P2.54mm_Vertical
- J17: value Conn_01x11_Female -> Conn_01x10_Female; footprint Connector_PinHeader_2.54mm:PinHeader_1x11_P2.54mm_Vertical -> Connector_PinSocket_2.54mm:PinSocket_1x10_P2.54mm_Vertical
- J8: footprint Connector_PinHeader_2.54mm:PinHeader_1x02_P2.54mm_Vertical -> Connector_PinSocket_2.54mm:PinSocket_1x02_P2.54mm_Vertical
- moved R4 19.2 mm to (21.6, 30.2)
- moved R7 18.9 mm to (19.1, 23.6), turned to 0 degrees
- moved C4 12.9 mm to (22.6, 35.8), turned to 0 degrees
- moved C3 12.0 mm to (34.3, 43.9), turned to 90 degrees
- moved R8 9.20 mm to (40.9, 50.8)
- moved U3 4.21 mm to (17.3, 29.2)
- moved J8 1.92 mm to (2.54, 29.0), turned to 0 degrees
- moved R3 1.82 mm to (6.86, 28.4), turned to 0 degrees
- moved J12 1.52 mm to (19.8, 19.1)
- moved SW2 1.38 mm to (39.6, 39.1)
- moved U1 0.83 mm to (42.9, 12.9)
- moved J11 0.39 mm to (43.5, 57.9)
- moved R2 0.31 mm to (12.2, 33.8)
Connections:
- J14 pad 2: 34 -> 23
- J17 pad 1: 23 -> 21
- J17 pad 10: +3V3 -> V_SWITCH
- J17 pad 2: 21 -> 19
- J17 pad 3: 19 -> 18:DHT22
- J17 pad 4: 18:DHT22 -> 5:onewire
- J17 pad 5: 5:onewire -> 0
- J17 pad 6: 0 -> 14:SCL
- J17 pad 7: 14:SCL -> 2:SDA
- J17 pad 8: 2:SDA -> GND
- J17 pad 9: GND -> +3V3
Routing:
- net GND: track 44.2 -> 420.2 mm, vias 0 -> 6
- net +3V3: track 40.3 -> 267.0 mm, vias 0 -> 6
- net V_SWITCH: track 3.22 -> 170.5 mm
- net RESET: track 0.00 -> 114.0 mm, vias 0 -> 5
- net 19: track 0.00 -> 105.3 mm, vias 0 -> 7
- net RX0: track 0.00 -> 89.2 mm, vias 0 -> 10
- net 21: track 0.00 -> 84.3 mm, vias 0 -> 5
- net 14:SCL: track 4.02 -> 81.3 mm, vias 0 -> 5
- net 23: track 0.00 -> 75.0 mm, vias 0 -> 4
- net Net-(C1-Pad1): track 0.45 -> 72.4 mm, vias 0 -> 3
- net 0: track 0.00 -> 71.1 mm, vias 0 -> 5
- net 5:onewire: track 0.00 -> 69.2 mm, vias 0 -> 1
- net 35: track 0.00 -> 67.9 mm, vias 0 -> 2
- net TX0: track 0.00 -> 67.2 mm, vias 0 -> 4
- net 18:DHT22: track 0.00 -> 67.0 mm
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Other:
- outline, holes or cut-outs redrawn

Commit message: update
Routing:
- net 21: track 84.3 -> 106.8 mm, vias 5 -> 6
- net 0: track 71.1 -> 87.4 mm, vias 5 -> 6
- net 14:SCL: track 81.3 -> 93.5 mm, vias 5 -> 8
- net 19: track 105.3 -> 99.9 mm
- net RX0: track 89.2 -> 92.7 mm
- net 23: track 75.0 -> 77.4 mm
- net +3V3: track 267.0 -> 268.7 mm
- net TX0: track 67.2 -> 68.4 mm
- net 2:SDA: track 64.2 -> 64.9 mm
- net GND: track 420.2 -> 420.7 mm
- net 18:DHT22: track 67.0 -> 67.4 mm, vias 0 -> 1

Commit message: update
Parts:
- moved J2 2.91 mm to (6.35, 67.8), turned to 0 degrees
- moved C1 2.48 mm to (45.2, 78.7), turned to 90 degrees
- moved C5 1.58 mm to (22.1, 69.3)
- moved J4 1.44 mm to (31.8, 62.0)
- moved C2 1.31 mm to (37.1, 68.1)
- moved J1 1.30 mm to (38.8, 76.5)
- moved S1 1.28 mm to (3.56, 37.4)
- moved Q2 1.15 mm to (7.62, 37.8)
- moved J13 1.08 mm to (2.29, 75.9)
- moved J6 1.05 mm to (26.6, 76.6)
- moved J18 0.33 mm to (13.0, 67.8)
Routing:
- net GND: track 420.7 -> 402.0 mm
- net +3V3: track 268.7 -> 260.6 mm, vias 6 -> 4
- net Net-(C1-Pad1): track 72.4 -> 66.1 mm, vias 3 -> 4
- net 4: track 56.8 -> 58.3 mm
- net 15: track 53.8 -> 55.3 mm
- net Net-(BT1-Pad1): track 46.9 -> 48.2 mm
- net Net-(Q2-Pad1): track 11.6 -> 12.6 mm
- net +5V: track 34.5 -> 33.7 mm
- net VIN: track 46.0 -> 46.8 mm, vias 0 -> 1
- net 12: track 65.1 -> 65.8 mm
- net Net-(S1-Pad2): track 41.3 -> 42.0 mm
Other:
- outline, holes or cut-outs redrawn

Commit message: update
Parts:
- moved J2 37.8 mm to (12.7, 30.5), turned to 180 degrees
Routing:
- net VIN: track 46.8 -> 75.2 mm, vias 1 -> 2
- net V_SWITCH: track 170.5 -> 183.1 mm
- net Net-(J16-Pad2): track 38.9 -> 41.2 mm, vias 3 -> 4
- net GND: track 402.0 -> 403.6 mm
- net 34: track 34.8 -> 35.9 mm
- net Net-(J8-Pad1): track 14.8 -> 15.4 mm
Other:
- board text added: "13"
- board text added: "OFF"
- board text added: "ON"
- board text added: "VS"
- board text added: "edgecollective.io/quahog"
- board text added: "ver 1.2"
- board text removed: "22"
- board text removed: "26"
- board text removed: "33"
- board text removed: "DTR"
- board text removed: "VIN"
- board text removed: "http://edgecollective.io/quahog"
- board text removed: "ver 0.1"

Commit message: update
Parts:
- moved C6 1.15 mm to (8.92, 63.6)
- moved C2 0.51 mm to (36.6, 67.8)
Routing:
- net +5V: track 33.7 -> 34.5 mm
Other:
- board text added: "26"
- board text added: "33"

Commit message: update
Parts:
- moved J16 6.37 mm to (47.0, 47.3)
Routing:
- net RESET: track 114.0 -> 122.9 mm, vias 5 -> 6
- net Net-(J16-Pad2): track 41.2 -> 47.6 mm, vias 4 -> 5
- net 19: track 99.9 -> 102.5 mm
- net 21: track 106.8 -> 107.6 mm

Commit message: update
Parts:
- J10, J4: footprint Pin_Headers:Pin_Header_Straight_1x07_Pitch2.54mm -> Connector_PinSocket_2.54mm:PinSocket_1x07_P2.54mm_Vertical
- J16, J2: footprint Connector_PinHeader_2.54mm:PinHeader_1x02_P2.54mm_Vertical -> Connector_PinSocket_2.54mm:PinSocket_1x02_P2.54mm_Vertical
- J3: footprint Connector_PinHeader_2.54mm:PinHeader_1x06_P2.54mm_Vertical -> Connector_PinSocket_2.54mm:PinSocket_1x06_P2.54mm_Vertical
- moved J16 2.23 mm to (45.4, 48.8), turned to 0 degrees
Routing:
- net V_SWITCH: track 182.6 -> 195.4 mm, vias 0 -> 2
- net RESET: track 122.9 -> 120.0 mm
- net 21: track 107.6 -> 104.8 mm, vias 6 -> 4
- net Net-(J16-Pad2): track 47.6 -> 50.0 mm
- net 19: track 102.5 -> 102.4 mm, vias 7 -> 5
Other:
- board text added: "3V"

Commit message: update
Other:
- board text added: "CR1220"
- board text added: "SSD1306"
Changed lines of the file:
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@@
   (general
     (thickness 1.6)
-    (drawings 97)
+    (drawings 99)
     (tracks 1072)
     (zones 0)
@@
     (descr "Through hole straight pin header, 1x04, 2.54mm pitch, single row")
     (tags "Through hole pin header THT 1x04 2.54mm single row")
-    (fp_text reference J5 (at 0.1016 -2.9098) (layer F.SilkS)
+    (fp_text reference J5 (at 0.8806 -2.2494) (layer F.SilkS)
       (effects (font (size 1 1) (thickness 0.15)))
     )
@@
     (fp_line (start 1.8 9.4) (end 1.8 -1.8) (layer F.CrtYd) (width 0.05))
     (fp_line (start 1.8 -1.8) (end -1.8 -1.8) (layer F.CrtYd) (width 0.05))
-    (fp_text user %R (at 0.0678 -2.9098) (layer F.Fab)
+    (fp_text user %R (at 0.8806 -2.3256) (layer F.Fab)
       (effects (font (size 1 1) (thickness 0.15)))
     )
@@
     )
   )
+  (gr_text CR1220 (at 23.622 45.6438 315) (layer F.SilkS)
+    (effects (font (size 0.8 0.8) (thickness 0.125)))
+  )
+  (gr_text SSD1306 (at 39.3954 28.9814) (layer F.SilkS)
+    (effects (font (size 0.8 0.8) (thickness 0.125)))
+  )
   (gr_text GND (at 17.0688 3.8354) (layer B.SilkS)
     (effects (font (size 0.5 0.5) (thickness 0.125)) (justify mirror))
@@
   (gr_line (start 0 0) (end 58 0) (layer Edge.Cuts) (width 0.2))
   (gr_circle (center 29 3.556) (end 30.521941 3.556) (layer Edge.Cuts) (width 0.15))
-  (gr_text 2 (at 32.9565 26.2382) (layer F.SilkS)
+  (gr_text 2 (at 32.8168 26.3144) (layer F.SilkS)
     (effects (font (size 0.8 0.8) (thickness 0.125)))
   )
