File: hog32a.kicad_pcb (KiCad board)
At the start: 2 copper layers, 58 x 82 mm, 46 parts, among them J1 REG:3V3, J10 Conn_01x07, J11 Conn_01x06_Male, J12 dht22, J13 Screw_Terminal_01x02, J14 Conn_01x09_Female, J15 Conn_01x05, J16 Conn_01x02_Male, J17 Conn_01x10_Female, J18 Barrel_Jack_Switch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

Commit message: update
Parts:
- added JP1: SolderJumper_2_Bridged, Jumper:SolderJumper-2_P1.3mm_Bridged_RoundedPad1.0x1.5mm, F.Cu at (18.8, 38.6)
- added JP2: SolderJumper_2_Open, Jumper:SolderJumper-2_P1.3mm_Open_RoundedPad1.0x1.5mm, F.Cu at (28.8, 58.1)
- J14: value Conn_01x09_Female -> Conn_01x10_Female; footprint Connector_PinSocket_2.54mm:PinSocket_1x09_P2.54mm_Vertical -> Connector_PinSocket_2.54mm:PinSocket_1x10_P2.54mm_Vertical
- moved J14 0.90 mm to (1.78, 47.9)
- moved C5 0.59 mm to (22.7, 69.4)
- moved J13 0.23 mm to (2.21, 76.2)
Connections:
- R2 pad 2: Net-(J16-Pad2) -> Net-(JP1-Pad2)
Routing:
- net VIN: track 75.2 -> 100.6 mm, vias 2 -> 4
- net V_SWITCH: track 195.4 -> 203.4 mm, vias 2 -> 3
- net Net-(JP1-Pad2): track 0.00 -> 7.98 mm, vias 0 -> 1
- net 34: track 35.9 -> 40.3 mm
- net Net-(J16-Pad2): track 50.0 -> 53.8 mm
- net Net-(S1-Pad2): track 42.0 -> 44.8 mm
- net 35: track 67.9 -> 70.1 mm
- net 12: track 65.8 -> 68.0 mm
- net RESET: track 120.0 -> 120.9 mm
- net 23: track 77.4 -> 78.3 mm
- net +3V3: track 260.3 -> 259.6 mm
- net +5V: track 34.5 -> 35.0 mm
- net Net-(C1-Pad1): track 66.1 -> 66.6 mm
- net 15: vias 2 -> 3
Other:
- board text added: "VER 1.2"
- board text added: "VIN"
- board text removed: "RTS"
- board text removed: "ver 1.2"
